File: kicad_files/hermes.kicad_sch (KiCad schematic)
At the start: 29 parts, among them J1 TYPE-C-31-M12_13, SW1 Mechanical_Switch, SW2 Mechanical_Switch, SW3 Mechanical_Switch, U1 BL24C256A-SFRC, U2 STM32F411CEU6, X1 ARM JTAG, Y1 7325-0800A2010-00

Commit message: Placing switches
Parts:
- added D10, D11, D12, D13, D14, D15, D16, D17, D18, D19, D20, D21, D22, D23, D24, D25, D26, D27, D28, D29, D30, D31, D32, D33, D34, D35, D36, D37, D38, D39, D4, D40, D41, D42, D43, D44, D45, D46, D47, D48, D49, D5, D50, D51, D52, D53, D54, D55, D56, D57, D58, D59, D6, D60, D61, D62, D63, D64, D65, D66, D7, D8, D9: 1N4148W, acheron_Components:D_SOD-123, symbol Device:D_Small
- added LED1: LED, acheron_Components:LED_THT_2.54mm, symbol acheron_Symbols:LED
- added SW10, SW11, SW12, SW13, SW14, SW15, SW18, SW19, SW20, SW21, SW22, SW23, SW24, SW25, SW26, SW27, SW28, SW29, SW32, SW33, SW34, SW35, SW36, SW37, SW38, SW39, SW4, SW40, SW41, SW42, SW43, SW48, SW49, SW5, SW50, SW51, SW52, SW53, SW54, SW55, SW56, SW57, SW58, SW6, SW60, SW7, SW72, SW76, SW8, SW9: Mechanical_Switch, acheron_MX_soldermask:MX100, symbol acheron_Symbols:Mechanical_Switch
- added SW16: Mechanical_Switch, acheron_MX_soldermask:MX200, symbol acheron_Symbols:Mechanical_Switch
- added SW17, SW30, SW71, SW73, SW75, SW77: Mechanical_Switch, acheron_MX_soldermask:MX150, symbol acheron_Symbols:Mechanical_Switch
- added SW31, SW62: Mechanical_Switch, acheron_MX_soldermask:MX175, symbol acheron_Symbols:Mechanical_Switch
- added SW44, SW47: Mechanical_Switch, acheron_MX_soldermask:MX225, symbol acheron_Symbols:Mechanical_Switch
- added SW45: Mechanical_Switch, acheron_MX_soldermask:MX_ISOEnter, symbol acheron_Symbols:Mechanical_Switch
- added SW46, SW61, SW63, SW64, SW65, SW67, SW68, SW69, SW70: Mechanical_Switch, acheron_MX_soldermask:MX125, symbol acheron_Symbols:Mechanical_Switch
- added SW59: Mechanical_Switch, acheron_MX_soldermask:MX275, symbol acheron_Symbols:Mechanical_Switch
- added SW66: Mechanical_Switch, acheron_MX_soldermask:MX625R, symbol acheron_Symbols:Mechanical_Switch
- added SW74: Mechanical_Switch, acheron_MX_soldermask:MX700R, symbol acheron_Symbols:Mechanical_Switch
Connections:
- net C0: now also SW17.1, SW31.1, SW46.2, SW47.1, SW61.1, SW63.1, SW71.1
- net C1: now also SW18.1, SW32.1, SW48.1, SW64.1, SW72.1
- net C2: now also SW19.1, SW33.1, SW49.1, SW65.1, SW73.1
- net R0: now also D10.1 (K), D11.1 (K), D12.1 (K), D13.1 (K), D14.1 (K), D15.1 (K), D4.1 (K), D5.1 (K), D6.1 (K), D7.1 (K), D8.1 (K), D9.1 (K)
- new net: D47.2 (A), SW49.2
- new net: D64.2 (A), SW68.2, SW75.2
- new net: D55.2 (A), SW57.2
- new net: D17.2 (A), SW18.2
- new net: D58.2 (A), SW60.2
- new net: D35.2 (A), SW36.2
- new net: D59.2 (A), SW63.2, SW71.2
- new net: D9.2 (A), SW9.2
- new net: D36.2 (A), SW37.2
- new net: D6.2 (A), SW6.2
- new net: D61.2 (A), SW65.2, SW73.2
- new net: D29.2 (A), SW30.2
- new net: D50.2 (A), SW52.2
- new net: D13.2 (A), SW13.2
- new net: D27.2 (A), SW28.2
- new net: D12.2 (A), SW12.2
- new net: D7.2 (A), SW7.2
- new net: D37.2 (A), SW38.2
- new net: D34.2 (A), SW35.2
- new net: D44.2 (A), SW45.2
- new net: D65.2 (A), SW69.2, SW76.2
- new net: D66.2 (A), SW70.2, SW77.2
- new net: D43.2 (A), SW44.2
- new net: D49.2 (A), SW51.2
- new net: D33.2 (A), SW34.2
- new net: D63.2 (A), SW67.2
- new net: D26.2 (A), SW27.2
- new net: D14.2 (A), SW14.2
- new net: D19.2 (A), SW20.2
- new net: D22.2 (A), SW23.2
- new net: D31.2 (A), SW32.2
- new net: D51.2 (A), SW53.2
- new net: D28.2 (A), SW29.2
- new net: D48.2 (A), SW50.2
- new net: D45.2 (A), SW47.2, SW61.2
- new net: D10.2 (A), SW10.2
- new net: D41.2 (A), SW42.2
- new net: D21.2 (A), SW22.2
- new net: D30.2 (A), SW31.2, SW46.1
- new net: D25.2 (A), SW26.2
- new net: D60.2 (A), SW64.2, SW72.2
- new net: D39.2 (A), SW40.2
- new net: D4.2 (A), SW4.2
- new net: D57.2 (A), SW59.2, SW62.2
- new net: D40.2 (A), SW41.2
- new net: D53.2 (A), SW55.2
- new net: D24.2 (A), SW25.2
- new net: D38.2 (A), SW39.2
- new net: D20.2 (A), SW21.2
- new net: D46.2 (A), SW48.2
- new net: D62.2 (A), SW66.2, SW74.2
- new net: D42.2 (A), SW43.2
- new net: D54.2 (A), SW56.2
- new net: D8.2 (A), SW8.2
- new net: D23.2 (A), SW24.2
- new net: D52.2 (A), SW54.2
- new net: D16.2 (A), SW17.2
- new net: D15.2 (A), SW15.2, SW16.2
- new net: D5.2 (A), SW5.2
- new net: D32.2 (A), SW33.2
- new net: D18.2 (A), SW19.2
- new net: D11.2 (A), SW11.2
- new net: D56.2 (A), SW58.2
- new net C10: SW11.1, SW27.1, SW41.1, SW57.1
- new net C11: SW12.1, SW28.1, SW42.1, SW58.1, SW67.1
- new net C12: SW13.1, SW29.1, SW43.1, SW59.1, SW62.1, SW68.1, SW75.1
- new net C13: SW14.1, SW44.1, SW69.1, SW76.1
- new net C14: SW15.1, SW16.1, SW30.1, SW45.1, SW60.1, SW70.1, SW77.1
- new net C3: SW20.1, SW34.1, SW4.1, SW50.1
- new net C4: SW21.1, SW35.1, SW5.1, SW51.1
- new net C5: SW22.1, SW36.1, SW52.1, SW6.1
- new net C6: SW23.1, SW37.1, SW53.1, SW66.1, SW7.1, SW74.1
- new net C7: SW24.1, SW38.1, SW54.1, SW8.1
- new net C8: SW25.1, SW39.1, SW55.1, SW9.1
- new net C9: SW10.1, SW26.1, SW40.1, SW56.1
- new net R1: D16.1 (K), D17.1 (K), D18.1 (K), D19.1 (K), D20.1 (K), D21.1 (K), D22.1 (K), D23.1 (K), D24.1 (K), D25.1 (K), D26.1 (K), D27.1 (K), D28.1 (K), D29.1 (K)
- new net R2: D30.1 (K), D31.1 (K), D32.1 (K), D33.1 (K), D34.1 (K), D35.1 (K), D36.1 (K), D37.1 (K), D38.1 (K), D39.1 (K), D40.1 (K), D41.1 (K), D42.1 (K), D43.1 (K), D44.1 (K)
- new net R3: D45.1 (K), D46.1 (K), D47.1 (K), D48.1 (K), D49.1 (K), D50.1 (K), D51.1 (K), D52.1 (K), D53.1 (K), D54.1 (K), D55.1 (K), D56.1 (K), D57.1 (K), D58.1 (K)
- new net R4: D59.1 (K), D60.1 (K), D61.1 (K), D62.1 (K), D63.1 (K), D64.1 (K), D65.1 (K), D66.1 (K)

Commit message: Name change to Raphael, move MCU and add RAPHAEL letters
Parts:
- added C1: 10u, Capacitor_SMD:C_0402_1005Metric, symbol Device:C_Small
- added C2: 100n, Capacitor_SMD:C_0402_1005Metric, symbol Device:C_Small
- added C3, C4: 1u, Capacitor_SMD:C_0805_2012Metric, symbol Device:C
- added C5: 10n, Capacitor_SMD:C_0402_1005Metric, symbol Device:C_Small
- added D1: 1N4148W, acheron_Components:D_SOD-123, symbol Device:D
- added D2: B5819W-SL, acheron_Components:D_SOD-123, symbol Device:D_Schottky
- added F1: nSMD100-16V, Fuse:Fuse_1206_3216Metric, symbol Device:Fuse
- added FB1: GZ2012D601TF, Inductor_SMD:L_0805_2012Metric, symbol Device:Ferrite_Bead_Small
- added J1: A1001WR-S-04P, acheron_Connectors:SM04B-SRSS-TB(LF)(SN)_mounting-reliefs, symbol Connector_Generic_MountingPin:Conn_01x04_MountingPin
- added Q1, Q2: 2N7002, Package_TO_SOT_SMD:SOT-23, symbol Transistor_FET:2N7002
- added R1: 330k, Resistor_SMD:R_0402_1005Metric, symbol Device:R_Small
- added R10: 10k, Resistor_SMD:R_0805_2012Metric, symbol Device:R_Small
- added R16, R17: 5.1k, Resistor_SMD:R_0402_1005Metric, symbol Device:R_Small
- added R2: 1M, Resistor_SMD:R_0402_1005Metric, symbol Device:R_Small
- added R3, R9: 10k, Resistor_SMD:R_0402_1005Metric, symbol Device:R_Small
- added R4, R5, R6: 100R, Resistor_SMD:R_0402_1005Metric, symbol Device:R_Small
- added R7, R8: 100k, Resistor_SMD:R_0805_2012Metric, symbol Device:R
- added SW1: K2-1187SQ-A4SW-06, acheron_Hardware:K2-1187SQ-A4SW-06, symbol Switch:SW_SPST
- added U1: USBLC6-2SC6, acheron_Components:SOT-23-6, symbol Power_Protection:USBLC6-2SC6
- added U2: SGM2007-3.3XN5/TR, acheron_Components:SOT-23-5, symbol acheron_Symbols:SGM2036
- renumbered C5 to C10, C6 to C11, C7 to C12, C8 to C13, C9 to C14, C10 to C15, C11 to C16, C1 to C6, C2 to C7, C3 to C8, C4 to C9, D8 to D10, D9 to D11, D10 to D12, D11 to D13, D12 to D14, D13 to D15, D14 to D16, D15 to D17, D16 to D18, D17 to D19, D18 to D20, D19 to D21, D20 to D22, D21 to D23, D22 to D24, D23 to D25, D24 to D26, D25 to D27, D26 to D28, D27 to D29, D1 to D3, D28 to D30, D29 to D31, D30 to D32, D31 to D33, D32 to D34, D33 to D35, D34 to D36, D35 to D37, D36 to D38, D37 to D39, D2 to D4, D38 to D40, D39 to D41, D40 to D42, D41 to D43, D42 to D44, D43 to D45, D44 to D46, D45 to D47, D46 to D48, D47 to D49, D3 to D5, D48 to D50, D49 to D51, D50 to D52, D51 to D53, D52 to D54, D53 to D55, D54 to D56, D55 to D57, D56 to D58, D57 to D59, D4 to D6, D58 to D60, D59 to D61, D60 to D62, D61 to D63, D62 to D64, D63 to D65, D64 to D66, D65 to D67, D66 to D68, D5 to D7, D6 to D8, D7 to D9, J1 to J2, R1 to R11, R2 to R12, R3 to R13, R4 to R14, R5 to R15, SW9 to SW10, SW10 to SW11, SW11 to SW12, SW12 to SW13, SW13 to SW14, SW14 to SW15, SW15 to SW16, SW16 to SW17, SW17 to SW18, SW18 to SW19, SW1 to SW2, SW19 to SW20, SW20 to SW21, SW21 to SW22, SW22 to SW23, SW23 to SW24, SW24 to SW25, SW25 to SW26, SW26 to SW27, SW27 to SW28, SW28 to SW29, SW2 to SW3, SW29 to SW30, SW30 to SW31, SW31 to SW32, SW32 to SW33, SW33 to SW34, SW34 to SW35, SW35 to SW36, SW36 to SW37, SW37 to SW38, SW38 to SW39, SW3 to SW4, SW39 to SW40, SW40 to SW41, SW41 to SW42, SW42 to SW43, SW43 to SW44, SW44 to SW45, SW45 to SW46, SW46 to SW47, SW47 to SW48, SW48 to SW49, SW4 to SW5, SW49 to SW50, SW50 to SW51, SW51 to SW52, SW52 to SW53, SW53 to SW54, SW54 to SW55, SW55 to SW56, SW56 to SW57, SW57 to SW58, SW58 to SW59, SW5 to SW6, SW59 to SW60, SW60 to SW61, SW61 to SW62, SW62 to SW63, SW63 to SW64, SW64 to SW65, SW65 to SW66, SW66 to SW67, SW67 to SW68, SW68 to SW69, SW6 to SW7, SW69 to SW70, SW70 to SW71, SW71 to SW72, SW72 to SW73, SW73 to SW74, SW74 to SW75, SW75 to SW76, SW76 to SW77, SW77 to SW78, SW7 to SW8, SW8 to SW9, U1 to U3, U2 to U4
Connections:
- net 3V3: now also C4.1, D2.2 (A), R8.1, SW1.1 (A), U2.5 (OUT)
- net 5V: now also C3.1, D2.1 (K), F1.1, J1.1 (Pin_1), R7.1, U2.1 (IN), U2.3 (EN)
- net BOOT0: now also C1.1, R1.1, R2.1, R3.2
- net D+: now also J1.3 (Pin_3), U1.3 (I/O2)
- net D-: now also J1.2 (Pin_2), U1.1 (I/O1)
- net GND: now also C1.2, C2.2, C3.2, C4.2, C5.1, FB1.2, J1.4 (Pin_4), J1.MP (MountPin), Q1.2 (S), Q2.2 (S), R10.2, R16.1, R17.2, R2.2, R7.2, R8.2, R9.1, U1.2 (GND), U2.2 (GND)
- net NRST: now also C2.1, R5.2
- net PB2/BOOT1: now also R10.1
- net VBUS: now reaches J2.A4 (VBUS)
- net VBUS: now also J2.B4 (VBUS), F1.2, U1.5 (VBUS)
- net at J2.A5 (CC1): now also R16.2
- net DBUS+: now reaches J2.A6 (D+)
- net DBUS+: now also J2.B6 (D+), U1.4 (I/O2)
- net DBUS-: now reaches J2.A7 (D-)
- net DBUS-: now also J2.B7 (D-), U1.6 (I/O1)
- net at J2.B5 (CC2): now also R17.1
- net GNDPWR: now reaches J2.S (SHIELD)
- net GNDPWR: now also FB1.1
- new net: Q1.1 (G), R4.2
- new net: Q1.3 (D), R3.1
- new net: D1.2 (A), R6.2, SW1.2 (B)
- new net: Q2.3 (D), R4.1, R5.1
- new net: C5.2, U2.4 (BP/FB)
- new net: Q2.1 (G), R6.1, R9.2
- new net: D1.1 (K), R1.2
- no-connect marks 1 -> 3
Other:
- note added: "3V3"
- note added: "HARD RESET"
- note added: "USB ESD"
- moved on the sheet: J2

Commit message: Place diodes and LEDs
Parts:
- added LED10, LED11, LED12, LED13, LED14, LED15, LED16, LED17, LED18, LED19, LED2, LED20, LED21, LED22, LED23, LED24, LED25, LED26, LED27, LED28, LED29, LED3, LED30, LED31, LED32, LED33, LED34, LED35, LED36, LED37, LED38, LED39, LED4, LED40, LED41, LED42, LED43, LED44, LED45, LED46, LED47, LED48, LED49, LED5, LED50, LED51, LED52, LED53, LED54, LED55, LED56, LED57, LED58, LED59, LED6, LED60, LED61, LED62, LED63, LED64, LED65, LED66, LED67, LED68, LED69, LED7, LED70, LED71, LED72, LED73, LED74, LED75, LED76, LED8, LED9: LED, acheron_Components:LED_THT_2.54mm, symbol acheron_Symbols:LED
- added Q3: AO3401A, Package_TO_SOT_SMD:SOT-23, symbol Transistor_FET:AO3401A
- added Q4, Q5: 2N7002, Package_TO_SOT_SMD:SOT-23, symbol Transistor_FET:2N7002
- added R18, R21: 10k, Resistor_SMD:R_0402_1005Metric, symbol Device:R_Small
- added R19, R20: 100, Resistor_SMD:R_0402_1005Metric, symbol Device:R_Small
- added R22, R23, R24, R25, R26, R27, R28, R29, R30, R31, R32, R33, R34, R35, R36, R37, R38, R39, R40, R41, R42, R43, R44, R45, R46, R47, R48, R49, R50, R51, R52, R53, R54, R55, R56, R57, R58, R59, R60, R61, R62, R63, R64, R65, R67, R68, R69, R70, R71, R72, R73, R74, R75, R76, R77, R78, R79, R81, R82, R83, R84, R85, R86, R87, R88, R89, R90: 1k, Resistor_SMD:R_0805_2012Metric, symbol Device:R_Small
- added R66: 100, Resistor_SMD:R_0805_2012Metric, symbol Device:R_Small
- added R80: 10k, Resistor_SMD:R_0805_2012Metric, symbol Device:R_Small
- C5: footprint Capacitor_SMD:C_0402_1005Metric -> Capacitor_SMD:C_0805_2012Metric; Manufacturer Part Number CL05B103KB5NNNC -> CL21B103KBANNNC; Package C0402 -> C0805; Specification 50V 10nF X7R ±10% 0402 MLCC -> 50V 10nF X7R ±10% 0805 MLCC; Vendor Part Number LCSC C15195 -> LCSC C1710
- LED1: now left out of the parts list
- SW46: footprint acheron_MX_soldermask:MX_ISOEnter -> acheron_MX_soldermask:MX_ISOEnter_Horizontal
Connections:
- net 5V: now also Q3.2 (S), R18.2
- net C0: now also SW64.2, SW72.2; no longer SW64.1, SW72.1
- net C2: now also SW20.2, SW50.2; no longer SW20.1, SW50.1
- net CAPS_INDICATOR: now also R66.1
- net GND: now also LED1.K, LED10.K, LED11.K, LED12.K, LED13.K, LED14.K, LED15.K, LED16.K, LED17.K, LED18.K, LED19.K, LED2.K, LED20.K, LED21.K, LED22.K, LED23.K, LED24.K, LED25.K, LED26.K, LED27.K, LED28.K, LED29.K, LED3.K, LED30.K, LED31.K, LED35.K, LED36.K, LED37.K, LED38.K, LED39.K, LED4.K, LED40.K, LED41.K, LED42.K, LED43.K, LED44.K, LED45.K, LED46.K, LED49.K, LED5.K, LED50.K, LED51.K, LED52.K, LED53.K, LED54.K, LED55.K, LED56.K, LED57.K, LED58.K, LED59.K, LED6.K, LED60.K, LED61.K, LED62.K, LED63.K, LED64.K, LED65.K, LED66.K, LED67.K, LED68.K, LED69.K, LED7.K, LED70.K, LED71.K, LED72.K, LED73.K, LED74.K, LED75.K, LED76.K, LED8.K, LED9.K, Q4.2 (S), Q5.2 (S), R21.1, R65.2, R80.1, R81.2, R82.2
- net LED_PWM: now also R20.1
- net at D49.2 (A): now also SW50.1; no longer SW50.2
- net at D20.2 (A): now also SW20.1; no longer SW20.2
- net at LED1.A: now also R22.2
- new net: LED32.A, LED47.A, LED48.A, Q3.3 (D), R22.1, R23.1, R24.1, R25.1, R26.1, R27.1, R28.1, R29.1, R30.1, R31.1, R32.1, R33.1, R34.1, R35.1, R36.1, R37.1, R38.1, R39.1, R40.1, R41.1, R42.1, R43.1, R44.1, R45.1, R46.1, R47.1, R48.1, R49.1, R50.1, R51.1, R52.1, R53.1, R54.1, R55.1, R56.1, R57.1, R58.1, R59.1, R60.1, R61.1, R62.1, R63.1, R64.1, R67.1, R68.1, R69.1, R70.1, R71.1, R72.1, R73.1, R74.1, R75.1, R76.1, R77.1, R78.1, R79.1, R83.1, R84.1, R85.1, R86.1, R87.1, R88.1, R89.1, R90.1
- new net: LED3.A, R24.2
- new net: LED26.A, R44.2
- new net: LED6.A, R27.2
- new net: LED30.A, R48.2
- new net: LED38.A, R56.2
- new net: LED37.A, R55.2
- new net: LED23.A, R41.2
- new net: LED58.A, R76.2
- new net: LED31.A, R49.2
- new net: LED54.A, R71.2
- new net: LED60.A, R78.2
- new net: D61.2 (A), SW64.1, SW72.1
- new net: Q5.1 (G), R66.2, R80.2
- new net: LED33.K, LED34.K, Q5.3 (D)
- new net: LED20.A, R38.2
- new net: LED35.A, R53.2
- new net: LED14.A, R35.2
- new net: LED75.A, LED76.A, R90.2
- new net: LED57.A, R75.2
- new net: LED51.A, R68.2
- new net: LED53.A, R70.2
- new net: LED55.A, R73.2
- new net: LED62.A, LED63.A, R83.2
- new net: LED49.A, R72.2
- new net: LED21.A, R39.2
- new net: LED5.A, R26.2
- new net: LED2.A, R23.2
- new net: Q4.3 (D), R18.1, R19.1
- new net: Q3.1 (G), R19.2
- new net: LED39.A, R57.2
- new net: LED15.A, LED16.A, R36.2
- new net: LED68.A, LED69.A, R86.2
- new net: LED18.A, R51.2
- new net: LED44.A, R62.2
- new net: LED41.A, R59.2
- new net: LED66.A, LED67.A, R85.2
- new net: LED71.A, LED72.A, R88.2
- new net: LED47.K, R81.1
- new net: LED32.K, R65.1
- new net: Q4.1 (G), R20.2, R21.2
- new net: LED4.A, R25.2
- new net: LED27.A, R45.2
- new net: LED12.A, R33.2
- new net: LED24.A, R42.2
- new net: LED22.A, R40.2
- new net: LED59.A, R77.2
- new net: LED50.A, R67.2
- new net: LED73.A, LED74.A, R89.2
- new net: LED48.K, R82.1
- new net: LED45.A, R63.2
- new net: LED61.A, R79.2
- new net: LED28.A, R46.2
- new net: LED56.A, R74.2
- new net: LED33.A, LED34.A, R52.2
- new net: LED42.A, R60.2
- new net: LED11.A, R32.2
- new net: LED7.A, R28.2
- new net: LED9.A, R30.2
- new net: LED10.A, R31.2
- new net: LED13.A, R34.2
- new net: LED19.A, R37.2
- new net: LED43.A, R61.2
- new net: LED64.A, LED65.A, R84.2
- new net: LED46.A, R64.2
- new net: LED36.A, R54.2
- new net: LED70.A, R87.2
- new net: LED40.A, R58.2
- new net: LED52.A, R69.2
- new net: LED25.A, R43.2
- new net: LED8.A, R29.2
- new net: LED17.A, R50.2
- new net: LED29.A, R47.2
Other:
- note added: "LED BACKLIGHT"
- moved on the sheet: SW20, SW50, SW64, SW72

Commit message: Finish routing; DRC pending
Parts:
- removed R10: 10k, Resistor_SMD:R_0805_2012Metric, symbol Device:R_Small
- removed R15: 0R, Resistor_SMD:R_0805_2012Metric, symbol Device:R_Small
- removed R78, R81: 1k, Resistor_SMD:R_0805_2012Metric, symbol Device:R_Small
- added J2: Conn_01x01, acheron_Connectors:PinHeader_1x3_staggered_P2.54mm_Vertical, symbol Connector_Generic:Conn_01x03
- added LED55: LED, acheron_Components:LED_THT_2.54mm, symbol acheron_Symbols:LED
- added R69: 1k, Resistor_SMD:R_0805_2012Metric, symbol Device:R_Small
- SW41: renamed from SW45; footprint acheron_MX_soldermask:MX225 -> acheron_MX_soldermask:MX225R
- renumbered D11 to D10, D12 to D11, D13 to D12, D14 to D13, D15 to D14, D16 to D15, D17 to D16, D20 to D17, D21 to D18, D22 to D19, D23 to D20, D24 to D21, D25 to D22, D26 to D23, D27 to D24, D28 to D25, D29 to D26, D30 to D27, D31 to D28, D33 to D29, D4 to D3, D34 to D30, D35 to D31, D36 to D32, D37 to D33, D38 to D34, D39 to D35, D40 to D36, D41 to D37, D42 to D38, D43 to D39, D5 to D4, D44 to D40, D45 to D41, D46 to D42, D47 to D43, D48 to D44, D49 to D45, D50 to D46, D51 to D47, D52 to D48, D53 to D49, D6 to D5, D54 to D50, D55 to D51, D56 to D52, D57 to D53, D58 to D54, D59 to D55, D60 to D56, D61 to D57, D62 to D58, D63 to D59, D7 to D6, D64 to D60, D65 to D61, D66 to D62, D67 to D63, D68 to D64, D3 to D65, D18 to D66, D32 to D67, D19 to D68, D8 to D7, D9 to D8, D10 to D9, J2 to J3, LED19 to LED17, LED20 to LED18, LED24 to LED19, LED6 to LED2, LED17 to LED20, LED18 to LED21, LED21 to LED22, LED22 to LED23, LED23 to LED24, LED2 to LED3, LED38 to LED32, LED39 to LED38, LED40 to LED39, LED3 to LED4, LED41 to LED40, LED32 to LED41, LED52 to LED49, LED4 to LED5, LED53 to LED50, LED49 to LED51, LED50 to LED52, LED51 to LED53, LED55 to LED56, LED56 to LED57, LED57 to LED58, LED58 to LED59, LED5 to LED6, LED59 to LED60, LED60 to LED61, LED61 to LED62, LED62 to LED63, LED63 to LED64, LED64 to LED65, LED65 to LED66, LED66 to LED67, LED67 to LED68, LED68 to LED69, LED69 to LED70, LED70 to LED71, LED71 to LED72, LED72 to LED73, LED73 to LED74, LED74 to LED75, LED75 to LED76, LED76 to LED77, R13 to R10, R14 to R13, R16 to R14, R17 to R15, R18 to R16, R19 to R17, R20 to R18, R21 to R19, R23 to R20, R24 to R21, R25 to R22, R26 to R23, R28 to R24, R29 to R25, R30 to R26, R31 to R27, R32 to R28, R33 to R29, R34 to R30, R35 to R31, R36 to R32, R22 to R33, R27 to R34, R39 to R35, R40 to R36, R41 to R37, R43 to R38, R44 to R39, R45 to R40, R46 to R41, R47 to R42, R48 to R43, R49 to R44, R50 to R45, R51 to R46, R37 to R47, R38 to R48, R42 to R49, R52 to R50, R53 to R51, R54 to R52, R55 to R53, R57 to R54, R58 to R55, R59 to R56, R65 to R57, R60 to R58, R61 to R59, R62 to R60, R63 to R61, R64 to R62, R56 to R63, R66 to R64, R67 to R65, R68 to R66, R71 to R67, R72 to R68, R73 to R70, R74 to R71, R75 to R72, R76 to R73, R77 to R74, R79 to R75, R80 to R76, R82 to R77, R69 to R78, R70 to R79, R84 to R80, R85 to R81, R86 to R82, R87 to R83, R88 to R84, R89 to R85, R90 to R86, R83 to R87, SW11 to SW10, SW12 to SW11, SW13 to SW12, SW14 to SW13, SW15 to SW14, SW16 to SW15, SW17 to SW16, SW20 to SW17, SW21 to SW18, SW22 to SW19, SW3 to SW2, SW23 to SW20, SW24 to SW21, SW25 to SW22, SW26 to SW23, SW27 to SW24, SW28 to SW25, SW29 to SW26, SW30 to SW27, SW31 to SW28, SW33 to SW29, SW4 to SW3, SW34 to SW30, SW35 to SW31, SW36 to SW32, SW37 to SW33, SW38 to SW34, SW39 to SW35, SW40 to SW36, SW41 to SW37, SW42 to SW38, SW43 to SW39, SW5 to SW4, SW44 to SW40, SW46 to SW42, SW48 to SW43, SW49 to SW44, SW50 to SW45, SW51 to SW46, SW52 to SW47, SW53 to SW48, SW54 to SW49, SW6 to SW5, SW55 to SW50, SW56 to SW51, SW57 to SW52, SW58 to SW53, SW59 to SW54, SW60 to SW55, SW61 to SW56, SW62 to SW57, SW63 to SW58, SW64 to SW59, SW7 to SW6, SW65 to SW60, SW66 to SW61, SW67 to SW62, SW68 to SW63, SW69 to SW64, SW70 to SW65, SW71 to SW66, SW72 to SW67, SW73 to SW68, SW74 to SW69, SW8 to SW7, SW75 to SW70, SW76 to SW71, SW77 to SW72, SW78 to SW73, SW2 to SW74, SW18 to SW75, SW32 to SW76, SW47 to SW77, SW19 to SW78, SW9 to SW8, SW10 to SW9
Connections:
- net 3V3: now also J2.1 (Pin_1)
- net C0: now also U4.27 (PB14)
- net C1: now also U4.31 (PA10)
- net C10: now also U4.17 (PA7)
- net C11: now also U4.15 (PA5)
- net C12: now also U4.11 (PA1)
- net C13: now also U4.3 (PC14_OSC32IN)
- net C14: now also U4.4 (PC15_OSC32OUT)
- net C2: now also U4.39 (PB3)
- net C3: now also U4.46 (PB9)
- net C4: now also U4.45 (PB8)
- net C5: now also U4.41 (PB5)
- net C6: now also U4.25 (PB12)
- net C7: now also U4.21 (B10)
- net C8: now also U4.19 (PB1)
- net C9: now also U4.18 (PB0)
- net CAPS_INDICATOR: now also U4.12 (PA2); no longer U4.19 (PB1)
- net GND: now also LED41.K, R33.2, R34.2, R47.2, R48.2, R49.2, R63.1, R78.2, R79.2, R87.2, J2.3 (Pin_3), LED55.K; no longer LED1.K, LED17.K, LED18.K, LED19.K, LED2.K, LED32.K, LED49.K, LED50.K, LED63.K, LED64.K, R57.2
- net PA9: now also J2.2 (Pin_2)
- net R0: now also U4.10 (PA0-WKUP); no longer D65.1 (K)
- net R1: now also U4.40 (PB4); no longer D66.1 (K), D68.1 (K)
- net R2: now also U4.2 (PC13); no longer D67.1 (K)
- net R3: now also U4.14 (PA4)
- net R4: now also U4.26 (PB13)
- net at LED47.A, LED48.A, Q3.3 (D)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: now also LED1.A, LED17.A, LED18.A, LED19.A, LED2.A, LED32.A, LED49.A, LED50.A, LED63.A, LED64.A, R57.1, R69.1; no longer LED41.A, R33.1, R34.1, R47.1, R48.1, R49.1, R63.1, R78.1, R79.1, R87.1
- net R7: now reaches U4.13 (PA3)
- net R7: now also D67.1 (K)
- net R6: now reaches U4.29 (PA8)
- net R6: now also D66.1 (K)
- net R8: now reaches U4.38 (PA15)
- net R8: now also D68.1 (K)
- net at R63.2: now also LED32.K; no longer LED32.A
- net at LED61.A: now also LED60.A, R74.2
- net at LED47.K: now also LED48.K, R77.1
- net RGB_3V3 renamed R5
- net R5: now also D65.1 (K)
- new net: LED2.K, R34.1
- new net: LED18.K, R48.1
- new net: LED50.K, R79.1
- new net: LED55.A, R69.2
- new net: LED63.K, LED64.K, R87.1
- new net: LED1.K, R33.1
- new net: LED41.A, R57.2
- new net: LED19.K, R49.1
- new net: LED17.K, R47.1
- new net: LED49.K, R78.1
- no-connect marks 3 -> 2
Other:
- title: Hermes PCB schematic -> Raphael PCB schematic
- moved on the sheet: D10, D11, D12, D13, D14, D15, D16, D17, D18, D19, D20, D21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

Commit message: Reset circuit, QoL
- Reset circuit was updated with a single-package double MOSFET 2N7002DW
- Quality of life tracing improvements
Parts:
- removed Q1, Q2: 2N7002, Package_TO_SOT_SMD:SOT-23, symbol Transistor_FET:2N7002
- added U2: (no value), symbol acheron_Symbols:2N7002DW
- renumbered LED35 to LED33, LED36 to LED34, LED37 to LED35, LED38 to LED36, LED39 to LED37, LED40 to LED38, LED41 to LED39, LED42 to LED40, LED43 to LED41, LED44 to LED42, LED45 to LED43, LED46 to LED44, LED33 to LED45, LED34 to LED46, Q3 to Q1, Q4 to Q2, Q5 to Q3, R51 to R50, R52 to R51, R53 to R52, R54 to R53, R55 to R54, R56 to R55, R57 to R56, R58 to R57, R59 to R58, R60 to R59, R61 to R60, R62 to R61, R50 to R62, R65 to R64, R66 to R65, R67 to R66, R68 to R67, R69 to R68, R70 to R69, R71 to R70, R72 to R71, R73 to R72, R74 to R73, R75 to R74, R64 to R75, U2 to U3, U3 to U4, U4 to U5
Connections:
- net GND: now also U2.1 (S), U2.4 (S)
- net at R4.2: now also R5.1, U2.6 (D)
- net at R3.1: now also U2.3 (D)
- net at R4.1: now also U2.5 (G); no longer R5.1
- net at R6.1, R9.2: now also U2.2 (G)
Other:
- moved on the sheet: LED1, LED10, LED11, LED12, LED13, LED14, LED15, LED16, LED17, LED18, LED19, LED2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
