File: kicad_files/raphael.kicad_sch (KiCad schematic)
At the start: 343 parts, among them J1 A1001WR-S-04P, J2 Conn_01x01, J3 TYPE-C-31-M12_13, Q1 AO3401A, Q2 2N7002, Q3 2N7002, SW1 K2-1187SQ-A4SW-06, SW10 Mechanical_Switch, SW11 Mechanical_Switch, SW12 Mechanical_Switch, SW13 Mechanical_Switch, SW14 Mechanical_Switch, SW15 Mechanical_Switch, SW16 Mechanical_Switch, SW17 Mechanical_Switch, SW18 Mechanical_Switch, SW19 Mechanical_Switch, SW2 Mechanical_Switch, SW20 Mechanical_Switch, SW21 Mechanical_Switch, SW22 Mechanical_Switch, SW23 Mechanical_Switch, SW24 Mechanical_Switch, SW25 Mechanical_Switch, SW26 Mechanical_Switch, SW27 Mechanical_Switch, SW28 Mechanical_Switch, SW29 Mechanical_Switch, SW3 Mechanical_Switch, SW30 Mechanical_Switch, SW31 Mechanical_Switch, SW32 Mechanical_Switch, SW33 Mechanical_Switch, SW34 Mechanical_Switch, SW35 Mechanical_Switch, SW36 Mechanical_Switch, SW37 Mechanical_Switch, SW38 Mechanical_Switch, SW39 Mechanical_Switch, SW4 Mechanical_Switch, SW40 Mechanical_Switch, SW41 Mechanical_Switch, SW42 Mechanical_Switch, SW43 Mechanical_Switch, SW44 Mechanical_Switch, SW45 Mechanical_Switch, SW46 Mechanical_Switch, SW47 Mechanical_Switch, SW48 Mechanical_Switch, SW49 Mechanical_Switch, SW5 Mechanical_Switch, SW50 Mechanical_Switch, SW51 Mechanical_Switch, SW52 Mechanical_Switch, SW53 Mechanical_Switch, SW54 Mechanical_Switch, SW55 Mechanical_Switch, SW56 Mechanical_Switch, SW57 Mechanical_Switch, SW58 Mechanical_Switch, SW59 Mechanical_Switch, SW6 Mechanical_Switch, SW60 Mechanical_Switch, SW61 Mechanical_Switch, SW62 Mechanical_Switch, SW63 Mechanical_Switch, SW64 Mechanical_Switch, SW65 Mechanical_Switch, SW66 Mechanical_Switch, SW67 Mechanical_Switch, SW68 Mechanical_Switch, SW69 Mechanical_Switch, SW7 Mechanical_Switch, SW70 Mechanical_Switch, SW71 Mechanical_Switch, SW72 Mechanical_Switch, SW73 Mechanical_Switch, SW74 Mechanical_Switch, SW75 Mechanical_Switch, SW76 Mechanical_Switch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

Commit message: Add label
Parts:
- added GR3, GR4: (no value), symbol Mechanical:MountingHole
- C1: value 10u -> (none); footprint Capacitor_SMD:C_0402_1005Metric -> (none)
- C10: value 10u -> (none); footprint acheron_Components:CP_EIA-3216-10_Kemet-I_Pad1.58x1.35mm_HandSolder -> (none); Manufacturer (none) -> AVX; Manufacturer Part Number (none) -> TAJA106K016RNJ; Specification (none) -> 10uF ±10% 16V CASE-A_3216 Tantalum Capacitor; Vendor Part Number (none) -> LCSC C7171
- C11: value 1u -> (none); footprint Capacitor_SMD:C_0402_1005Metric -> (none); Manufacturer Part Number (none) -> CL05A475MP5NRNC; Specification MLCC 10V or more -> 10V 4.7uF X5R ±20% 0402 MLCC; Vendor Part Number (none) -> LCSC C23733
- C12: value 10n -> (none); footprint Capacitor_SMD:C_0402_1005Metric -> (none); Manufacturer (none) -> Samsung; Manufacturer Part Number (none) -> CL05B103KB5NNNC; Specification MLCC 10V or more -> 50V 10nF X7R ±10% 0402 MLCC; Vendor Part Number (none) -> LCSC C15195
- C13, C14: value 16p -> (none); footprint Capacitor_SMD:C_0402_1005Metric -> (none); Manufacturer (none) -> Guangdong Fenghua Advanced Tech; Manufacturer Part Number (none) -> 0402CG150J500NT; Specification (none) -> 50V 10nF X7R ±10% 0402 MLCC; Vendor Part Number (none) -> LCSC C1548
- C15, C7, C8, C9: value 100n -> (none); footprint Capacitor_SMD:C_0402_1005Metric -> (none); Manufacturer (none) -> Samsung; Manufacturer Part Number (none) -> CL05B104KB54PNC; Specification MLCC 10V or more -> 50V 100nF X7R ±10% 0402 MLCC; Vendor Part Number (none) -> LCSC C307331
- C16: value 4.7u -> (none); footprint Capacitor_SMD:C_0402_1005Metric -> (none); Manufacturer (none) -> Samsung; Manufacturer Part Number (none) -> CL05A475MP5NRNC; Specification (none) -> 10V 4.7uF X5R ±20% 0402 MLCC
- C2: value 100n -> (none); footprint Capacitor_SMD:C_0402_1005Metric -> (none)
- C3, C4: value 1u -> (none); footprint Capacitor_SMD:C_0805_2012Metric -> (none)
- C5: value 10n -> (none); footprint Capacitor_SMD:C_0805_2012Metric -> (none)
- C6: value 100n -> (none); footprint Capacitor_SMD:C_0402_1005Metric -> (none); Manufacturer (none) -> Samsung; Manufacturer Part Number (none) -> CL05B104KB54PNC; Specification (none) -> 50V 100nF X7R ±10% 0402 MLCC; Vendor Part Number (none) -> LCSC C307331
- D1: value 1N4148W -> (none); footprint acheron_Components:D_SOD-123 -> (none); Specification Small-signal switching diodes -> 400mW 1μA@75V 150mA SOD-123 small-signal witching diode
- D10, D11, D12, D13, D14, D15, D16, D17, D18, D19, D20, D21, D22, D23, D24, D25, D26, D27, D28, D29, D3, D30, D31, D32, D33, D34, D35, D36, D37, D38, D39, D4, D40, D41, D42, D43, D44, D45, D46, D47, D48, D49, D5, D50, D51, D52, D53, D54, D55, D56, D57, D58, D59, D6, D60, D61, D62, D63, D64, D65, D66, D67, D68, D7, D8, D9: value 1N4148W -> (none); footprint acheron_Components:D_SOD-123 -> (none); Specification (none) -> 400mW 1μA@75V 150mA SOD-123 small-signal witching diode
- D2: value B5819W-SL -> (none); footprint acheron_Components:D_SOD-123 -> (none)
- F1: value nSMD100-16V -> (none); footprint Fuse:Fuse_1206_3216Metric -> (none)
- FB1: value GZ2012D601TF -> (none); footprint Inductor_SMD:L_0805_2012Metric -> (none)
- GR1: value Hermes huge logo -> (none); footprint hermes_library:hermes_logo_56.9x84mm -> (none)
- GR2: value Hermes plated logo -> (none); footprint hermes_library:hermes_plated_logo_12x17.7mm -> (none)
- J1: value A1001WR-S-04P -> (none); footprint acheron_Connectors:SM04B-SRSS-TB(LF)(SN)_mounting-reliefs -> (none)
- J2: renamed from J3; value TYPE-C-31-M12_13 -> (none); footprint acheron_Connectors:TYPE-C-31-M-12 -> (none); Manufacturer (none) -> Korean Hroparts; Manufacturer Part Number (none) -> TYPE-C-31-M-12; Specification (none) -> 250mA 16-pin female USB Type-C SMD connector; Vendor Part Number (none) -> LCSC C165948
- LED1, LED10, LED11, LED12, LED13, LED14, LED15, LED16, LED17, LED18, LED19, LED2, LED20, LED21, LED22, LED23, LED24, LED25, LED26, LED27, LED28, LED29, LED3, LED30, LED31, LED32, LED33, LED34, LED35, LED36, LED37, LED38, LED39, LED4, LED40, LED41, LED42, LED43, LED44, LED45, LED46, LED47, LED48, LED49, LED5, LED50, LED51, LED52, LED53, LED54, LED55, LED56, LED57, LED58, LED59, LED6, LED60, LED61, LED62, LED63, LED64, LED65, LED66, LED67, LED68, LED69, LED7, LED70, LED71, LED72, LED73, LED74, LED75, LED76, LED77, LED8, LED9: value LED -> (none); footprint acheron_Components:LED_THT_2.54mm -> (none)
- Q1: value AO3401A -> (none); footprint Package_TO_SOT_SMD:SOT-23 -> (none)
- Q2, Q3: value 2N7002 -> (none); footprint Package_TO_SOT_SMD:SOT-23 -> (none)
- R1: value 330k -> (none); footprint Resistor_SMD:R_0402_1005Metric -> (none)
- R10: value 10k -> (none); footprint Resistor_SMD:R_0805_2012Metric -> (none); Manufacturer (none) -> Uniroyal; Manufacturer Part Number (none) -> 0402WGF1002TCE; Package R0805 -> R0402; Specification (none) -> ±1% 1/16W Thick Film Resistors 50V 0402; Vendor Part Number (none) -> LCSC C25744
- R11, R12: value 1.5k -> (none); footprint Resistor_SMD:R_0402_1005Metric -> (none); Manufacturer (none) -> Uniroyal; Manufacturer Part Number (none) -> 0402WGF4701TCE; Specification (none) -> ±1% 1/16W Thick Film Resistors 50V 0402; Vendor Part Number (none) -> LCSC C25900
- R13: value 1.5k -> (none); footprint Resistor_SMD:R_0402_1005Metric -> (none); Manufacturer (none) -> Uniroyal; Manufacturer Part Number (none) -> 0402WGF1501TCE; Specification (none) -> ±1% 1/16W Thick Film Resistors 50V 0402; Vendor Part Number (none) -> LCSC C25867
- R14, R15: value 5.1k -> (none); footprint Resistor_SMD:R_0402_1005Metric -> (none)
- R16, R19, R3, R9: value 10k -> (none); footprint Resistor_SMD:R_0402_1005Metric -> (none)
- R17, R18: value 100 -> (none); footprint Resistor_SMD:R_0402_1005Metric -> (none)
- R2: value 1M -> (none); footprint Resistor_SMD:R_0402_1005Metric -> (none)
- R20, R21, R22, R23, R24, R25, R26, R27, R28, R29, R30, R31, R32, R33, R34, R35, R36, R37, R38, R39, R40, R41, R42, R43, R44, R45, R46, R47, R48, R49, R50, R51, R52, R53, R54, R55, R56, R57, R58, R59, R60, R61, R62, R63, R64, R65, R66, R67, R68, R69, R70, R71, R72, R73, R74, R77, R78, R79, R80, R81, R82, R83, R84, R85, R86, R87: value 1k -> (none); footprint Resistor_SMD:R_0805_2012Metric -> (none)
- R4, R5, R6: value 100R -> (none); footprint Resistor_SMD:R_0402_1005Metric -> (none)
- R7, R8: value 100k -> (none); footprint Resistor_SMD:R_0805_2012Metric -> (none)
- R75: value 100 -> (none); footprint Resistor_SMD:R_0805_2012Metric -> (none)
- R76: value 10k -> (none); footprint Resistor_SMD:R_0805_2012Metric -> (none)
- SW1: value K2-1187SQ-A4SW-06 -> (none); footprint acheron_Hardware:K2-1187SQ-A4SW-06 -> (none)
- SW10, SW11, SW12, SW13, SW14, SW15, SW17, SW18, SW19, SW2, SW20, SW21, SW22, SW23, SW24, SW25, SW26, SW27, SW29, SW3, SW30, SW31, SW32, SW33, SW34, SW35, SW36, SW37, SW38, SW39, SW4, SW40, SW44, SW45, SW46, SW47, SW48, SW49, SW5, SW50, SW51, SW52, SW53, SW54, SW56, SW6, SW68, SW7, SW72, SW74, SW78, SW8, SW9: value Mechanical_Switch -> (none); footprint acheron_MX_soldermask:MX100 -> (none)
- SW16: value Mechanical_Switch -> (none); footprint acheron_MX_soldermask:MX200 -> (none)
- SW28, SW67, SW69, SW71, SW73, SW75: value Mechanical_Switch -> (none); footprint acheron_MX_soldermask:MX150 -> (none)
- SW41: value Mechanical_Switch -> (none); footprint acheron_MX_soldermask:MX225R -> (none)
- SW42: value Mechanical_Switch -> (none); footprint acheron_MX_soldermask:MX_ISOEnter_Horizontal -> (none)
- SW43: value Mechanical_Switch -> (none); footprint acheron_MX_soldermask:MX225 -> (none)
- SW55: value Mechanical_Switch -> (none); footprint acheron_MX_soldermask:MX275 -> (none)
- SW57, SW59, SW60, SW61, SW63, SW64, SW65, SW66, SW77: value Mechanical_Switch -> (none); footprint acheron_MX_soldermask:MX125 -> (none)
- SW58, SW76: value Mechanical_Switch -> (none); footprint acheron_MX_soldermask:MX175 -> (none)
- SW62: value Mechanical_Switch -> (none); footprint acheron_MX_soldermask:MX625R -> (none)
- SW70: value Mechanical_Switch -> (none); footprint acheron_MX_soldermask:MX700R -> (none)
- U1: value USBLC6-2SC6 -> (none); footprint acheron_Components:SOT-23-6 -> (none)
- U2: Specification (none) -> Dual N-channel enhancement mode MOSFET
- U3: value SGM2007-3.3XN5/TR -> (none); footprint acheron_Components:SOT-23-5 -> (none)
- U4: value BL24C256A-SFRC -> (none); footprint acheron_Components:TSSOP-8_4.4x3mm_P0.65mm -> (none); Specification (none) -> TSSOP-8 non-volatile 256Kb (32K x 8) I2C EEPROM
- U5: value STM32F411CEU6 -> (none); footprint acheron_Components:STM_UFQFPN-48_LQFP-48-1EP_7x7mm_P0.5mm_HandSoldering_ThermalReliefs -> (none); Specification (none) -> 32-bit ARM Cortex-M0+ 128kBytes flash microcontroller
- X1: value ARM JTAG -> (none); footprint acheron_Connectors:PinHeader_2x5_P2.54mm_Vertical_Staggered -> (none)
- X2: renamed from J2; value Conn_01x01 -> (none); footprint acheron_Connectors:PinHeader_1x3_staggered_P2.54mm_Vertical -> (none)
- Y1: value 7325-0800A2010-00 -> (none); footprint acheron_Components:Crystal_SMD_3225-4Pin_3.2x2.5mm -> (none); Specification (none) -> 8MHz 3225-4P oscillator crystal
Connections:
- net GND: now also R79.1; no longer R79.2
- net at LED1.A, LED17.A, LED18.A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: now also R84.2; no longer R84.1
- net at LED50.K: now also R79.2; no longer R79.1
- net at LED72.A, LED73.A: now also R84.1; no longer R84.2
Other:
- moved on the sheet: R79

Commit message: Organize schematic, preparing for release
Parts:
- C1: value (none) -> 10u; footprint (none) -> Capacitor_SMD:C_0402_1005Metric
- C10: value (none) -> 10u; footprint (none) -> acheron_Components:CP_EIA-3216-10_Kemet-I_Pad1.58x1.35mm_HandSolder
- C11, C16: value (none) -> 4.7u; footprint (none) -> Capacitor_SMD:C_0402_1005Metric
- C12: value (none) -> 10n; footprint (none) -> Capacitor_SMD:C_0402_1005Metric
- C13, C14: value (none) -> 16p; footprint (none) -> Capacitor_SMD:C_0402_1005Metric
- C15, C2, C6, C7, C8, C9: value (none) -> 100n; footprint (none) -> Capacitor_SMD:C_0402_1005Metric
- C3, C4: value (none) -> 1u; footprint (none) -> Capacitor_SMD:C_0805_2012Metric
- C5: value (none) -> 10n; footprint (none) -> Capacitor_SMD:C_0805_2012Metric
- D1, D10, D11, D12, D13, D14, D15, D16, D17, D18, D19, D20, D21, D22, D23, D24, D25, D26, D27, D28, D29, D3, D30, D31, D32, D33, D34, D35, D36, D37, D38, D39, D4, D40, D41, D42, D43, D44, D45, D46, D47, D48, D49, D5, D50, D51, D52, D53, D54, D55, D56, D57, D58, D59, D6, D60, D61, D62, D63, D64, D65, D66, D67, D68, D7, D8, D9: value (none) -> 1N4148W; footprint (none) -> acheron_Components:D_SOD-123
- D2: value (none) -> B5819W-SL; footprint (none) -> acheron_Components:D_SOD-123
- F1: value (none) -> nSMD100-16V; footprint (none) -> Fuse:Fuse_1206_3216Metric
- FB1: value (none) -> GZ2012D601TF; footprint (none) -> Inductor_SMD:L_0805_2012Metric
- GR1: value (none) -> Raphael huge logo; footprint (none) -> raphael_library:raphael_logo_56.9x84mm
- GR2: value (none) -> Raphael plated logo; footprint (none) -> raphael_library:raphael_plated_logo_12x17.7mm
- GR3: value (none) -> Rapahel letters; footprint (none) -> raphael_library:raphael_logo_letters_41x2.5mm
- GR4: value (none) -> Rapahel label; footprint (none) -> raphael_library:raphael_label_191x3mm
- J1: value (none) -> A1001WR-S-04P; footprint (none) -> acheron_Connectors:SM04B-SRSS-TB(LF)(SN)_mounting-reliefs
- J2: value (none) -> TYPE-C-31-M-12; footprint (none) -> acheron_Connectors:TYPE-C-31-M-12
- LED1, LED10, LED11, LED12, LED13, LED14, LED15, LED16, LED17, LED18, LED19, LED2, LED20, LED21, LED22, LED23, LED24, LED25, LED26, LED27, LED28, LED29, LED3, LED30, LED31, LED32, LED33, LED34, LED35, LED36, LED37, LED38, LED39, LED4, LED40, LED41, LED42, LED43, LED44, LED45, LED46, LED47, LED48, LED49, LED5, LED50, LED51, LED52, LED53, LED54, LED55, LED56, LED57, LED58, LED59, LED6, LED60, LED61, LED62, LED63, LED64, LED65, LED66, LED67, LED68, LED69, LED7, LED70, LED71, LED72, LED73, LED74, LED75, LED76, LED77, LED8, LED9: value (none) -> LED; footprint (none) -> acheron_Components:LED_THT_2.54mm
- Q1: value (none) -> AO3401A; footprint (none) -> Package_TO_SOT_SMD:SOT-23
- Q2, Q3: value (none) -> 2N7002; footprint (none) -> Package_TO_SOT_SMD:SOT-23
- R1: value (none) -> 330k; footprint (none) -> Resistor_SMD:R_0402_1005Metric
- R10, R16, R19, R3, R9: value (none) -> 10k; footprint (none) -> Resistor_SMD:R_0402_1005Metric
- R11, R12: value (none) -> 4.7k; footprint (none) -> Resistor_SMD:R_0402_1005Metric
- R13: value (none) -> 1.5k; footprint (none) -> Resistor_SMD:R_0402_1005Metric
- R14, R15: value (none) -> 5.1k; footprint (none) -> Resistor_SMD:R_0402_1005Metric
- R17, R18: value (none) -> 100; footprint (none) -> Resistor_SMD:R_0402_1005Metric
- R2: value (none) -> 1M; footprint (none) -> Resistor_SMD:R_0402_1005Metric
- R20, R21, R22, R23, R24, R25, R26, R27, R28, R29, R30, R31, R32, R33, R34, R35, R36, R37, R38, R39, R40, R41, R42, R43, R44, R45, R46, R47, R48, R49, R50, R51, R52, R53, R54, R55, R56, R57, R58, R59, R60, R61, R62, R63, R64, R65, R66, R67, R68, R69, R70, R71, R72, R73, R74, R77, R78, R79, R80, R81, R82, R83, R84, R85, R86, R87: value (none) -> 1k; footprint (none) -> Resistor_SMD:R_0805_2012Metric
- R4, R5, R6: value (none) -> 100R; footprint (none) -> Resistor_SMD:R_0402_1005Metric
- R7, R8: value (none) -> 100k; footprint (none) -> Resistor_SMD:R_0805_2012Metric
- R75: value (none) -> 100R; footprint (none) -> Resistor_SMD:R_0805_2012Metric
- R76: value (none) -> 10k; footprint (none) -> Resistor_SMD:R_0805_2012Metric
- SW1: value (none) -> K2-1187SQ-A4SW-06; footprint (none) -> acheron_Hardware:K2-1187SQ-A4SW-06
- SW10, SW11, SW12, SW13, SW14, SW15, SW17, SW18, SW19, SW2, SW20, SW21, SW22, SW23, SW24, SW25, SW26, SW27, SW29, SW3, SW30, SW31, SW32, SW33, SW34, SW35, SW36, SW37, SW38, SW39, SW4, SW40, SW44, SW45, SW46, SW47, SW48, SW49, SW5, SW50, SW51, SW52, SW53, SW54, SW56, SW6, SW68, SW7, SW72, SW74, SW78, SW8, SW9: value (none) -> Mechanical_Switch; footprint (none) -> acheron_MX_soldermask:MX100
- SW16: value (none) -> Mechanical_Switch; footprint (none) -> acheron_MX_soldermask:MX200
- SW28, SW67, SW69, SW71, SW73, SW75: value (none) -> Mechanical_Switch; footprint (none) -> acheron_MX_soldermask:MX150
- SW41: value (none) -> Mechanical_Switch; footprint (none) -> acheron_MX_soldermask:MX225R
- SW42: value (none) -> Mechanical_Switch; footprint (none) -> acheron_MX_soldermask:MX_ISOEnter_Horizontal
- SW43: value (none) -> Mechanical_Switch; footprint (none) -> acheron_MX_soldermask:MX225
- SW55: value (none) -> Mechanical_Switch; footprint (none) -> acheron_MX_soldermask:MX275
- SW57, SW59, SW60, SW61, SW63, SW64, SW65, SW66, SW77: value (none) -> Mechanical_Switch; footprint (none) -> acheron_MX_soldermask:MX125
- SW58, SW76: value (none) -> Mechanical_Switch; footprint (none) -> acheron_MX_soldermask:MX175
- SW62: value (none) -> Mechanical_Switch; footprint (none) -> acheron_MX_soldermask:MX625R
- SW70: value (none) -> Mechanical_Switch; footprint (none) -> acheron_MX_soldermask:MX700R
- U1: value (none) -> USBLC6-2SC6; footprint (none) -> acheron_Components:SOT-23-6
- U2: value (none) -> 2N7002DW; footprint (none) -> acheron_Components:SOT-363_SC-70-6
- U3: value (none) -> SGM2007-3.3XN5/TR; footprint (none) -> acheron_Components:SOT-23-5
- U4: value (none) -> BL24C256A-SFRC; footprint (none) -> acheron_Components:TSSOP-8_4.4x3mm_P0.65mm
- U5: value (none) -> STM32F411CEU6; footprint (none) -> acheron_Components:STM_UFQFPN-48_LQFP-48-1EP_7x7mm_P0.5mm_HandSoldering_ThermalReliefs
- X1: value (none) -> ARM JTAG; footprint (none) -> acheron_Connectors:PinHeader_2x5_P2.54mm_Vertical_Staggered
- X2: footprint (none) -> acheron_Connectors:PinHeader_1x3_staggered_P2.54mm_Vertical
- Y1: value (none) -> 7325-0800A2010-00; footprint (none) -> acheron_Components:Crystal_SMD_3225-4Pin_3.2x2.5mm
Other:
- note added: "GRAPHICS"
- note added: "USB"
- moved on the sheet: C1, C10, C11, C12, C13, C14, C15, C16, C2, C3, C4, C5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

Commit message: Edit metadata, release
Other:
- note added: "SWITCH MATRIX"
Changed lines of the file:
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@@
     (stroke (width 0) (type solid) (color 0 0 0 0))
+  )
+  (polyline (pts (xy 412.75 762) (xy 412.75 736.6))
+    (stroke (width 1.27) (type dash) (color 0 0 0 0))
   )
   (polyline (pts (xy 533.4 552.45) (xy 635 552.45))
@@
   (wire (pts (xy 165.735 573.405) (xy 167.005 573.405))
     (stroke (width 0) (type default) (color 0 0 0 0))
+  )
+  (polyline (pts (xy 412.75 736.6) (xy 514.35 736.6))
+    (stroke (width 1.27) (type dash) (color 0 0 0 0))
   )
   (wire (pts (xy 142.24 107.95) (xy 142.24 109.22))
@@
     (effects (font (size 7.62 7.62) (thickness 1.524) bold italic) (justify right bottom))
   )
+  (text "SWITCH MATRIX" (at 508 757.555 180)
+    (effects (font (size 7.62 7.62) (thickness 1.524) bold italic) (justify right bottom))
+  )

Commit message: Edit component metadata
Parts:
- R75: value 100R -> (none); footprint Resistor_SMD:R_0805_2012Metric -> (none); Manufacturer Part Number 0402WGF1000TCE -> 0805W8F1000T5E; Package R0402 -> R0805; Specification ±1% 1/16W Thick Film Resistors 50V 0402 -> ±1% 186W Thick Film Resistors 150V 0805; Vendor Part Number LCSC C25076 -> LCSC C17408
- R76: value 10k -> (none); footprint Resistor_SMD:R_0805_2012Metric -> (none); Manufacturer Part Number 0402WGF1002TCE -> 0805W8F1002T5E; Package R0402 -> R0805; Specification ±1% 1/16W Thick Film Resistors 50V 0402 -> ±1% 1/8W Thick Film Resistors 150V 0805; Vendor Part Number LCSC C25744 -> LCSC C17414
- U4: value BL24C256A-SFRC -> (none); footprint acheron_Components:TSSOP-8_4.4x3mm_P0.65mm -> (none); Vendor Part Number LCSC C691875 (https://lcsc.com/product-detail/EEPROM_BL-Sha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 -> LCSC C110276
- X2: value (none) -> EXTRA_PINS
Changed lines of the file:
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@@
   (title_block
     (title "Raphael PCB schematic")
-    (date "2022-04-09")
-    (rev "v1.0.1")
+    (date "2022-04-10")
+    (rev "v1.0.2")
     (company "AcheronProject")
     (comment 1 "Designed by Gondolindrim")
@@
       (effects (font (size 1.27 1.27)) (justify right))
     )
-    (property "Value" "10k" (id 1) (at 149.86 1022.9849 0)
+    (property "Value" "" (id 1) (at 149.86 1022.9849 0)
       (effects (font (size 1.27 1.27)) (justify right))
     )
-    (property "Footprint" "Resistor_SMD:R_0805_2012Metric" (id 2) (at 151.765 1022.35 0)
+    (property "Footprint" "" (id 2) (at 151.765 1022.35 0)
       (effects (font (size 1.27 1.27)) hide)
     )
@@
       (effects (font (size 1.27 1.27)) hide)
     )
-    (property "Package" "R0402" (id 5) (at 151.765 1022.35 0)
-      (effects (font (size 1.27 1.27)) hide)
-    )
     (property "Manufacturer" "Uniroyal" (id 6) (at 151.765 1022.35 0)
       (effects (font (size 1.27 1.27)) hide)
     )
-    (property "Manufacturer Part Number" "0402WGF1002TCE" (id 7) (at 161.9758 1022.35 0)
+    (property "Manufacturer Part Number" "0805W8F1002T5E" (id 7) (at 161.9758 1022.35 0)
       (effects (font (size 1.27 1.27)) hide)
     )
-    (property "Vendor Part Number" "LCSC C25744" (id 8) (at 151.765 1022.35 0)
+    (property "Vendor Part Number" "LCSC C17414" (id 8) (at 151.765 1022.35 0)
       (effects (font (size 1.27 1.27)) hide)
     )
-    (property "Specification" "±1% 1/16W Thick Film Resistors 50V 0402" (id 9) (at 151.765 1022.35 0)
+    (property "Specification" "±1% 1/8W Thick Film Resistors 150V 0805" (id 9) (at 151.765 1022.35 0)
       (effects (font (size 1.27 1.27)) hide)
     )
@@
     (in_bom yes) (on_board yes) (fields_autoplaced)
     (property "Reference" "R75" (id 0) (at 145.415 1009.65 90))
-    (property "Value" "100R" (id 1) (at 145.415 1012.19 90))
-    (property "Footprint" "Resistor_SMD:R_0805_2012Metric" (id 2) (at 145.415 1016 0)
+    (property "Value" "" (id 1) (at 145.415 1012.19 90))
+    (property "Footprint" "" (id 2) (at 145.415 1016 0)
       (effects (font (size 1.27 1.27)) hide)
     )
@@
       (effects (font (size 1.27 1.27)) hide)
     )
-    (property "Package" "R0402" (id 4) (at 145.415 1016 0)
+    (property "Package" "R0805" (id 4) (at 145.415 1016 0)
       (effects (font (size 1.27 1.27)) hide)
     )
@@
       (effects (font (size 1.27 1.27)) hide)
     )
-    (property "Manufacturer Part Number" "0402WGF1000TCE" (id 6) (at 145.415 1005.7892 0)
+    (property "Manufacturer Part Number" "0805W8F1000T5E" (id 6) (at 145.415 1005.7892 0)
       (effects (font (size 1.27 1.27)) hide)
     )
-    (property "Vendor Part Number" "LCSC C25076" (id 7) (at 145.415 1016 0)
+    (property "Vendor Part Number" "LCSC C17408" (id 7) (at 145.415 1016 0)
       (effects (font (size 1.27 1.27)) hide)
     )
-    (property "Specification" "±1% 1/16W Thick Film Resistors 50V 0402" (id 8) (at 145.415 1016 0)
+    (property "Specification" "±1% 186W Thick Film Resistors 150V 0805" (id 8) (at 145.415 1016 0)
       (effects (font (size 1.27 1.27)) hide)
     )
@@
       (effects (font (size 1.27 1.27)) (justify left))
     )
-    (property "Value" "" (id 1) (at 161.29 101.5999 0)
+    (property "Value" "EXTRA_PINS" (id 1) (at 161.29 101.5999 0)
       (effects (font (size 1.27 1.27)) (justify left))
     )
@@
     (in_bom yes) (on_board yes)
     (property "Reference" "U4" (id 0) (at 53.975 50.8 0))
-    (property "Value" "BL24C256A-SFRC" (id 1) (at 47.625 53.34 0))
-    (property "Footprint" "acheron_Components:TSSOP-8_4.4x3mm_P0.65mm" (id 2) (at 57.15 60.96 0)
+    (property "Value" "" (id 1) (at 47.625 53.34 0))
+    (property "Footprint" "" (id 2) (at 57.15 60.96 0)
       (effects (font (size 1.27 1.27)) hide)
     )
@@
       (effects (font (size 1.27 1.27)) hide)
     )
-    (property "Vendor Part Number" "LCSC C691875 (https://lcsc.com/product-detail/EEPROM_BL-Shanghai-Belling-BL24C256A-NTRC_C691875.html)" (id 8) (at 57.15 60.96 0)
-      (effects (font (size 1.27 1.27)) hide)
-    )
-    (property "Description" "" (id 9) (at 57.15 60.96 0)
+    (property "Vendor Part Number" "LCSC C110276" (id 8) (at 57.15 60.96 0)
       (effects (font (size 1.27 1.27)) hide)
     )
